File: untitled.kicad_sch (KiCad schematic)
At the start: 13 parts, among them J3 Conn_01x01_Pin, J4 Conn_01x01_Pin, J5 Conn_01x01_Pin, J6 Conn_01x01_Pin, J7 Conn_01x01_Pin, J8 Conn_01x01_Pin, J9 ECE05US05, K1 RT314A12, U11 ALDP112, U12 ALDP112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

Commit message: WIP
Parts:
- J3, J4, J5, J6, J7, J8: footprint Connector_Pin:Pin_D1.4mm_L8.5mm_W2.8mm_FlatFork -> 1289:KEYSTONE_1289
Changed lines of the file:
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@@
       (effects (font (size 1.27 1.27)))
     )
-    (property "Footprint" "Connector_Pin:Pin_D1.4mm_L8.5mm_W2.8mm_FlatFork" (at 26.67 137.16 0)
+    (property "Footprint" "1289:KEYSTONE_1289" (at 26.67 137.16 0)
       (effects (font (size 1.27 1.27)) hide)
     )
@@
       (effects (font (size 1.27 1.27)) (justify left))
     )
-    (property "Footprint" "Connector_Pin:Pin_D1.4mm_L8.5mm_W2.8mm_FlatFork" (at 151.13 144.78 0)
+    (property "Footprint" "1289:KEYSTONE_1289" (at 151.13 144.78 0)
       (effects (font (size 1.27 1.27)) hide)
     )
@@
       (effects (font (size 1.27 1.27)))
     )
-    (property "Footprint" "Connector_Pin:Pin_D1.4mm_L8.5mm_W2.8mm_FlatFork" (at 314.96 27.94 0)
+    (property "Footprint" "1289:KEYSTONE_1289" (at 314.96 27.94 0)
       (effects (font (size 1.27 1.27)) hide)
     )
@@
       (effects (font (size 1.27 1.27)))
     )
-    (property "Footprint" "Connector_Pin:Pin_D1.4mm_L8.5mm_W2.8mm_FlatFork" (at 321.31 90.17 0)
+    (property "Footprint" "1289:KEYSTONE_1289" (at 321.31 90.17 0)
       (effects (font (size 1.27 1.27)) hide)
     )
@@
       (effects (font (size 1.27 1.27)))
     )
-    (property "Footprint" "Connector_Pin:Pin_D1.4mm_L8.5mm_W2.8mm_FlatFork" (at 193.04 25.4 0)
+    (property "Footprint" "1289:KEYSTONE_1289" (at 193.04 25.4 0)
       (effects (font (size 1.27 1.27)) hide)
     )
@@
       (effects (font (size 1.27 1.27)))
     )
-    (property "Footprint" "Connector_Pin:Pin_D1.4mm_L8.5mm_W2.8mm_FlatFork" (at 20.32 123.19 0)
-      (effects (font (size 1.27 1.27)) hide)
-    )
+    (property "Footprint" "1289:KEYSTONE_1289" (at 20.32 123.19 0)
+      (effects (font (size 1.27 1.27)) hide)
+    )

Commit message: WIP
Parts:
- removed J9: ECE05US05, CONN5_05US05_XPP, symbol ECE05:ECE05US05
- added D2, D4, D5, D8: 1N4001, Diode_THT:D_DO-41_SOD81_P7.62mm_Horizontal, symbol Diode:1N4001
- added U2: ~, ECE05:ECE10, symbol ECE05:ECE10
- F1: value Fuse -> Schurter FRT 250T 7100.1009.13; footprint Fuse:Fuse_Bourns_MF-RG700 -> 1289:FRT 250T
- J3, J4, J5, J6, J7, J8: value Conn_01x01_Pin -> TE 160650-2
Connections:
- net +12VA: now also D2.1 (K), D4.1 (K), D5.1 (K), D8.1 (K), U2.4 (+Vout)
- net FA10_CTRL: now also D8.2 (A)
- net FA7_CTRL: now also D2.2 (A)
- net FA8_CTRL: now also D4.2 (A)
- net FA9_CTRL: now also D5.2 (A)
- net GND1: now also U2.3 (-Vout)
- net N: now also J8.1 (Pin_1), U2.1 (ACN); no longer J7.1 (Pin_1)
- net PH: now also U2.2 (ACL)
- net PH_PRE_FUSE: now reaches F1.1
- net PH_PRE_FUSE: now also J7.1 (Pin_1); no longer J8.1 (Pin_1)
- no-connect marks 2 -> 1
Other:
- moved on the sheet: J8
