File: open-control-board.kicad_sch (KiCad schematic)
At the start: 127 parts, among them CN1 Service boiler fill sensor, CN10 LCC Port, CN2 Water tank level switch, CN3 NTC Service Boiler, CN4 NTC Brew Boiler, CN5 Service boiler relay, CN6 Conn_02x04_Counter_Clockwise, CN7 Brew Switch, CN8 12V Separate Supply, CN9 Brew boiler relay, J1 USB_B_Micro, J10 Conn_01x04_Pin, J11 Conn_01x04_Pin, J12 Conn_02x06_Odd_Even, J13 Conn_02x05_Odd_Even, J14 Conn_02x04_Odd_Even, J15 Conn_02x05_Odd_Even, J16 USB_B_Micro, J5 BM04B-SRSS-TB(LF)(SN), Q1 AO3401A, Q2 AO3401A, Q3 AO3401A, Q4 AO3401A, Q5 AO3401A, SW1 SW_Push, SW2 SW_Push, SW3 SW_Push, SW4 SW_Push, U10 FDC1004, U15 STPIC6C595TTR, U16 STPIC6C595TTR, U2 MCP7940N-xSN, U2 RP2040, U3 ESP32-S3-WROOM-1, U4 W25Q16JVUXIQ, U6 TPS82130, U7 TXB0108DQSR, U8 ADS1115IDGS, Y1 XYDBPCNANF-12MHZ, Y3 YSX1610SK, 9 pF

Commit message: WIP
Parts:
- C13, C14, C15, C16, C17, C18, C19, C20, C21, C22, C24, C26, C29, C9: LCSC C960916 -> C307331
- C25, C27: LCSC C782176 -> C45783
- C28, C33: LCSC C2803388 -> C13585
- C28: value 22 uF, 10V, X5R -> 22 uF, 6.3V, X5R; LCSC C86295 -> C59461
- FB1, FB2: footprint PCM_Ferrite_SMD_AKL:Ferrite_0402_1005Metric -> PCM_Ferrite_SMD_AKL:Ferrite_0603_1608Metric; LCSC C480821 -> C1002
- R14, R7: LCSC C4288031 -> C17168
Changed lines of the file:
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@@
       (effects (font (size 1.27 1.27)) hide)
     )
-    (property "LCSC" "C960916" (at 320.04 273.05 0)
+    (property "LCSC" "C307331" (at 320.04 273.05 0)
       (effects (font (size 1.27 1.27)) hide)
     )
@@
       (effects (font (size 1.27 1.27)) hide)
     )
-    (property "LCSC" "C960916" (at 144.78 289.56 0)
+    (property "LCSC" "C307331" (at 144.78 289.56 0)
       (effects (font (size 1.27 1.27)) hide)
     )
@@
       (effects (font (size 1.27 1.27)) hide)
     )
-    (property "Footprint" "PCM_Ferrite_SMD_AKL:Ferrite_0402_1005Metric" (at 313.69 266.192 90)
+    (property "Footprint" "PCM_Ferrite_SMD_AKL:Ferrite_0603_1608Metric" (at 313.69 266.192 90)
       (effects (font (size 1.27 1.27)) hide)
     )
@@
       (effects (font (size 1.27 1.27)) hide)
     )
-    (property "LCSC" "C480821" (at 313.69 267.97 0)
+    (property "LCSC" "C1002" (at 313.69 267.97 0)
       (effects (font (size 1.27 1.27)) hide)
     )
@@
       (effects (font (size 1.27 1.27)) hide)
     )
-    (property "Footprint" "PCM_Ferrite_SMD_AKL:Ferrite_0402_1005Metric" (at 313.69 277.622 90)
+    (property "Footprint" "PCM_Ferrite_SMD_AKL:Ferrite_0603_1608Metric" (at 313.69 277.622 90)
       (effects (font (size 1.27 1.27)) hide)
     )
@@
       (effects (font (size 1.27 1.27)) hide)
     )
-    (property "LCSC" "C480821" (at 313.69 279.4 0)
+    (property "LCSC" "C1002" (at 313.69 279.4 0)
       (effects (font (size 1.27 1.27)) hide)
     )
@@
       (effects (font (size 1.27 1.27)) hide)
     )
-    (property "LCSC" "C4288031" (at 577.85 181.61 0)
+    (property "LCSC" "C17168" (at 577.85 181.61 0)
       (effects (font (size 1.27 1.27)) hide)
     )
@@
       (effects (font (size 1.27 1.27)) hide)
     )
-    (property "LCSC" "C782176" (at 204.47 81.28 0)
+    (property "LCSC" "C45783" (at 204.47 81.28 0)
       (effects (font (size 1.27 1.27)) hide)
     )
@@
       (effects (font (size 1.27 1.27)) hide)
     )
-    (property "LCSC" "C960916" (at 337.82 86.36 0)
+    (property "LCSC" "C307331" (at 337.82 86.36 0)
       (effects (font (size 1.27 1.27)) hide)
     )
@@
       (effects (font (size 1.27 1.27)) hide)
     )
-    (property "LCSC" "C2803388" (at 307.34 273.05 0)
+    (property "LCSC" "C13585" (at 307.34 273.05 0)
       (effects (font (size 1.27 1.27)) hide)
     )
@@
       (effects (font (size 1.27 1.27)) hide)
     )
-    (property "LCSC" "C782176" (at 204.47 22.86 0)
+    (property "LCSC" "C45783" (at 204.47 22.86 0)
       (effects (font (size 1.27 1.27)) hide)
     )
@@
       (effects (font (size 1.27 1.27)) hide)
     )
-    (property "LCSC" "C960916" (at 327.66 41.91 0)
+    (property "LCSC" "C307331" (at 327.66 41.91 0)
       (effects (font (size 1.27 1.27)) hide)
     )
@@
       (effects (font (size 1.27 1.27)) hide)
     )
-    (property "LCSC" "C782176" (at 220.98 90.17 0)
+    (property "LCSC" "C45783" (at 220.98 90.17 0)
       (effects (font (size 1.27 1.27)) hide)
     )
@@
       (effects (font (size 1.27 1.27)) hide)
     )
-    (property "LCSC" "C960916" (at 327.66 67.31 0)
+    (property "LCSC" "C307331" (at 327.66 67.31 0)
       (effects (font (size 1.27 1.27)) hide)
     )
@@
       (effects (font (size 1.27 1.27)) hide)
     )
-    (property "LCSC" "C960916" (at 327.66 57.15 0)
+    (property "LCSC" "C307331" (at 327.66 57.15 0)
       (effects (font (size 1.27 1.27)) hide)
     )
@@
       (effects (font (size 1.27 1.27)) hide)
     )
-    (property "LCSC" "C4288031" (at 577.85 179.07 0)
+    (property "LCSC" "C17168" (at 577.85 179.07 0)
       (effects (font (size 1.27 1.27)) hide)
     )
@@
       (effects (font (size 1.27 1.27)) hide)
     )
-    (property "LCSC" "C782176" (at 220.98 31.75 0)
+    (property "LCSC" "C45783" (at 220.98 31.75 0)
       (effects (font (size 1.27 1.27)) hide)
     )
@@
       (effects (font (size 1.27 1.27)) hide)
     )
-    (property "LCSC" "C2803388" (at 140.97 81.28 0)
+    (property "LCSC" "C13585" (at 140.97 81.28 0)
       (effects (font (size 1.27 1.27)) hide)
     )
@@
       (effects (font (size 1.27 1.27)) hide)
     )
-    (property "LCSC" "C960916" (at 327.66 46.99 0)
+    (property "LCSC" "C307331" (at 327.66 46.99 0)
       (effects (font (size 1.27 1.27)) hide)
     )
@@
       (effects (font (size 1.27 1.27)) hide)
     )
-    (property "LCSC" "C960916" (at 426.72 35.56 0)
+    (property "LCSC" "C307331" (at 426.72 35.56 0)
       (effects (font (size 1.27 1.27)) hide)
     )
@@
       (effects (font (size 1.27 1.27)) hide)
     )
-    (property "LCSC" "C2803388" (at 140.97 22.86 0)
+    (property "LCSC" "C13585" (at 140.97 22.86 0)
       (effects (font (size 1.27 1.27)) hide)
     )
@@
       (effects (font (size 1.27 1.27)) hide)
     )
-    (property "LCSC" "C960916" (at 335.28 76.2 0)
+    (property "LCSC" "C307331" (at 335.28 76.2 0)
       (effects (font (size 1.27 1.27)) hide)
     )
@@
       (effects (font (size 1.27 1.27)) hide)
     )
-    (property "LCSC" "C960916" (at 563.88 36.83 0)
+    (property "LCSC" "C307331" (at 563.88 36.83 0)
       (effects (font (size 1.27 1.27)) hide)
     )
@@
       (effects (font (size 1.27 1.27)) hide)
     )
-    (property "LCSC" "C960916" (at 321.31 100.33 0)
+    (property "LCSC" "C307331" (at 321.31 100.33 0)
       (effects (font (size 1.27 1.27)) hide)
     )
@@
       (effects (font (size 1.27 1.27)) hide)
     )
-    (property "LCSC" "C960916" (at 327.66 52.07 0)
+    (property "LCSC" "C307331" (at 327.66 52.07 0)
       (effects (font (size 1.27 1.27)) hide)
     )
@@
       (effects (font (size 1.27 1.27)))
     )
-    (property "Value" "22 uF, 10V, X5R" (at 575.3036 26.67 90)
+    (property "Value" "22 uF, 6.3V, X5R" (at 575.3036 26.67 90)
       (effects (font (size 1.27 1.27)))
     )
@@
       (effects (font (size 1.27 1.27)) hide)
     )
-    (property "LCSC" "C86295" (at 575.31 30.48 0)
+    (property "LCSC" "C59461" (at 575.31 30.48 0)
       (effects (font (size 1.27 1.27)) hide)
     )
@@
       (effects (font (size 1.27 1.27)) hide)
     )
-    (property "LCSC" "C960916" (at 327.66 62.23 0)
+    (property "LCSC" "C307331" (at 327.66 62.23 0)
       (effects (font (size 1.27 1.27)) hide)
     )
@@
       (effects (font (size 1.27 1.27)) hide)
     )
-    (property "LCSC" "C960916" (at 314.96 100.33 0)
+    (property "LCSC" "C307331" (at 314.96 100.33 0)
       (effects (font (size 1.27 1.27)) hide)
     )

Commit message: Added possibility to select CN10 levels via solder jumpers
Parts:
- removed BT1: Battery_Cell, BK-885:BAT_BK-885, symbol Device:Battery_Cell
- removed C2, C7: 11 pF, Capacitor_SMD:C_0402_1005Metric, symbol Device:C_Small
- removed C26: 100 nF, 50V, X7R, Capacitor_SMD:C_0402_1005Metric, symbol Device:C_Small
- removed U2: MCP7940N-xSN, Package_SO:SOP-8_3.76x4.96mm_P1.27mm, symbol Timer_RTC:MCP7940N-xSN
- removed Y3: YSX1610SK, 9 pF, SMD1610-2P:SMD1610-2P, symbol Device:Crystal
- added J18: Conn_01x03_Pin, Connector_PinHeader_2.54mm:PinHeader_1x03_P2.54mm_Vertical_SMD_Pin1Left, symbol Connector:Conn_01x03_Pin
- added JP10, JP11, JP9: SolderJumper_3_Bridged12, Jumper:SolderJumper-3_P1.3mm_Bridged2Bar12_RoundedPad1.0x1.5mm_NumberLabels, symbol Jumper:SolderJumper_3_Bridged12
- added JP12: SolderJumper_2_Open, Jumper:SolderJumper-2_P1.3mm_Open_RoundedPad1.0x1.5mm, symbol Jumper:SolderJumper_2_Open
- added Q6, Q7: 2N7002, Package_TO_SOT_SMD:SOT-23, symbol PCM_Transistor_MOSFET_AKL:2N7002
- added R41, R42, R43, R44: 10K, Resistor_SMD:R_0402_1005Metric, symbol Device:R_Small
- J1, J16: footprint Connector_USB:USB_Micro-B_Molex-105133-0031 -> U-D-M5DS-W-3:U-D-M5DS-W-3; LCSC C586226 -> C2909202
- JP4, JP5, JP6: footprint Jumper:SolderJumper-3_P1.3mm_Bridged2Bar12_Pad1.0x1.5mm_NumberLabels -> Jumper:SolderJumper-3_P1.3mm_Bridged2Bar12_RoundedPad1.0x1.5mm_NumberLabels
- SW1, SW2, SW3, SW4: footprint Button_Switch_SMD:SW_SPST_B3S-1000 -> ul_PTS815-SJM-250-SMTR-LFS:SW4_PTS815 SJM 250 SMTR LFS_CNK; Comment Hand solder -> (none); LCSC (none) -> C2689510
- U7: value TXB0108DQSR -> TXB0108PWR; footprint Package_SON:USON-20_2x4mm_P0.4mm -> Package_SO:TSSOP-20_4.4x6.5mm_P0.65mm; LCSC C427057 -> C53406
Connections:
- net +3V3: now also JP9.1 (A), Q6.1 (G), Q7.1 (G), R41.1, R43.1; no longer CN10.6 (Pin_6)
- net +5V: now also JP9.3 (B), R42.1, R44.1
- net CN10_UART_RX: now also R5.2, JP11.2 (C), JP12.1 (A); no longer R6.2, U2.28 (GPIO17), U3.10 (GPIO17/U1TXD/ADC2_CH6)
- net CN10_UART_TX: now also JP10.2 (C), Q6.2 (S), R41.2; no longer R5.2
- net GND: now also J18.3 (Pin_3)
- net ESP32_CTS0: no longer names the net of U3.9 (GPIO16/U0CTS/ADC2_CH5/XTAL_32K_N)
- net ESP32_RTS0: no longer names the net of U3.8 (GPIO15/U0RTS/ADC2_CH4/XTAL_32K_P)
- net ESP32_RXD0: no longer names the net of U3.36 (U0RXD/GPIO44/CLK_OUT2)
- net ESP32_RXD0: now also J18.1 (Pin_1)
- net ESP32_TXD0: no longer names the net of U3.37 (U0TXD/GPIO43/CLK_OUT1)
- net ESP32_TXD0: now also J18.2 (Pin_2)
- net RTC_MFP renamed GP15
- new net: JP10.3 (B), Q6.3 (D), R42.2
- new net: JP11.3 (B), Q7.2 (S), R43.2
- new net: JP12.2 (B), Q7.3 (D), R44.2
- new net: CN10.6 (Pin_6), JP9.2 (C)
- new net CN10_UART_RX_SHIFT_SEL: JP11.1 (A), U2.28 (GPIO17), U3.10 (GPIO17/U1TXD/ADC2_CH6)
- new net CN10_UART_TX_SHIFT_SEL: JP10.1 (A), R6.2
- no-connect marks 18 -> 20
Other:
- note added: "CN10 5V Level Shifter (Opt.)"
- note removed: "9 pF = (C25 * C26) / (C25 + C26) + CStray CStray is assumed to 3.5 pF C25 = C26 = 11 pF"
- note removed: "RTC (Optional)"

Commit message: WIP
Parts:
- removed JP10, JP11: SolderJumper_3_Bridged12, Jumper:SolderJumper-3_P1.3mm_Bridged2Bar12_RoundedPad1.0x1.5mm_NumberLabels, symbol Jumper:SolderJumper_3_Bridged12
- removed JP12: SolderJumper_2_Open, Jumper:SolderJumper-2_P1.3mm_Open_RoundedPad1.0x1.5mm, symbol Jumper:SolderJumper_2_Open
- removed Q3, Q4, Q5: AO3401A, Package_TO_SOT_SMD:SOT-23, symbol PCM_Transistor_MOSFET_AKL:BSS215P
- removed Q6, Q7: 2N7002, Package_TO_SOT_SMD:SOT-23, symbol PCM_Transistor_MOSFET_AKL:2N7002
- removed R41, R42, R43, R44: 10K, Resistor_SMD:R_0402_1005Metric, symbol Device:R_Small
- added JP13: SolderJumper_3_Bridged12, Jumper:SolderJumper-3_P1.3mm_Bridged2Bar12_RoundedPad1.0x1.5mm_NumberLabels, symbol Jumper:SolderJumper_3_Bridged12
- added Q11, Q4, Q6: DMN63D8LDW, PCM_Package_TO_SOT_SMD_AKL:SOT-363_SC-70-6, symbol PCM_Transistor_MOSFET_AKL:DMN63D8LDW
- added Q3, Q5: Q_PMOS-E_DUAL_Generic_SEP_S1G1D2S2G2D1, PCM_Package_TO_SOT_SMD_AKL:Vishay_PowerPAK_SC70-6L_Dual, symbol PCM_Transistor_MOSFET_AKL:Q_PMOS-E_DUAL_Generic_SEP_S1G1D2S2G2D1
- added R49, R50: 10K, Resistor_SMD:R_0402_1005Metric, symbol Device:R_Small
- added RN1, RN2: 10K, PCM_Resistor_SMD_AKL:R_Array_Concave_4x0402, symbol PCM_Resistor_US_AKL:R_4x0402_Sep_Convex
Connections:
- net +3V3: now also J12.1 (Pin_1), JP13.1 (A), Q11.2 (G1), Q11.5 (G2), Q4.2 (G1), Q6.2 (G1), Q6.5 (G2), R49.1, RN1.7 (R2.2), RN1.8 (R1.2), RN2.5 (R4.2), RN2.6 (R3.2); no longer C28.1, FB1.2
- net +5V: now also JP13.3 (B); no longer J12.1 (Pin_1)
- net ADS1115_RDY: now also Q4.1 (S1), R49.2; no longer U8.2 (ALERT/RDY)
- net AGND: now also U8.1 (ADDR)
- net AVCC: now also R50.1, RN2.7 (R2.2), RN2.8 (R1.2)
- net CN10_UART_RX: now also Q11.3 (D2), RN1.3 (R3.1)
- net CN10_UART_RX_SHIFT_SEL: now also Q11.4 (S2), RN1.2 (R2.1)
- net CN10_UART_TX: now also Q11.1 (S1), RN1.1 (R1.1)
- net CN10_UART_TX_SHIFT_SEL: now also Q11.6 (D1), RN1.4 (R4.1)
- net GND: no longer U8.1 (ADDR)
- net INT_SCL: now also Q6.4 (S2), RN2.4 (R4.1); no longer U8.10 (SCL)
- net INT_SDA: now also Q6.1 (S1), RN2.3 (R3.1); no longer U8.9 (SDA)
- net VOUT_1: now also Q5.3 (D2)
- net VOUT_1_GATE: now also Q5.5 (G2)
- net VOUT_2: now also Q3.6 (D1)
- net VOUT_2_GATE: now also Q3.2 (G1)
- net VOUT_3: now also Q3.3 (D2)
- net VOUT_3_GATE: now also Q3.5 (G2)
- net at JP6.2 (C), R30.1: now also Q3.4 (S2)
- net at JP5.2 (C), R29.1: now also Q3.1 (S1)
- net at JP4.2 (C), R28.1: now also Q5.4 (S2)
- net CN10_UART_VCC: now reaches CN10.6 (Pin_6), JP9.2 (C)
- net CN10_UART_VCC: now also RN1.5 (R4.2), RN1.6 (R3.2)
- new net: C28.1, FB1.2, JP13.2 (C)
- new net ADS1115_RDY_AVCC: Q4.6 (D1), R50.2, U8.2 (ALERT/RDY)
- new net INT_SCL_AVCC: Q6.3 (D2), RN2.2 (R2.1), U8.10 (SCL)
- new net INT_SDA_AVCC: Q6.6 (D1), RN2.1 (R1.1), U8.9 (SDA)
- no-connect marks 20 -> 23
Other:
- note added: "CN10 UART Level Shifter"
- note removed: "CN10 5V Level Shifter (Opt.)"
- moved on the sheet: JP9

Commit message: WIP
Parts:
- Q11, Q4, Q6: LCSC (none) -> C211422
Changed lines of the file:
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@@
       (effects (font (size 1.27 1.27)) hide)
     )
+    (property "LCSC" "C211422" (at 162.56 275.59 0)
+      (effects (font (size 1.27 1.27)) hide)
+    )
     (pin "1")
     (pin "2")
@@
       (effects (font (size 1.27 1.27)) hide)
     )
+    (property "LCSC" "C211422" (at 403.86 283.21 0)
+      (effects (font (size 1.27 1.27)) hide)
+    )
     (pin "1")
     (pin "2")
@@
       (effects (font (size 1.27 1.27)) hide)
     )
+    (property "LCSC" "C211422" (at 166.37 326.39 0)
+      (effects (font (size 1.27 1.27)) hide)
+    )
     (pin "1")
     (pin "2")
@@
       (effects (font (size 1.27 1.27)) hide)
     )
+    (property "LCSC" "C211422" (at 405.13 349.25 0)
+      (effects (font (size 1.27 1.27)) hide)
+    )
     (pin "1")
     (pin "2")
@@
       (effects (font (size 1.27 1.27)) hide)
     )
+    (property "LCSC" "C211422" (at 405.13 367.03 0)
+      (effects (font (size 1.27 1.27)) hide)
+    )
     (pin "1")
     (pin "2")
@@
       (effects (font (size 1.27 1.27)) hide)
     )
+    (property "LCSC" "C211422" (at 405.13 320.04 0)
+      (effects (font (size 1.27 1.27)) hide)
+    )

Commit message: WIP
Parts:
- removed R14, R15, R16, R25, R3, R38, R39, R4, R40: 480R, 500mW, Resistor_SMD:R_0805_2012Metric, symbol Device:R_Small
- added C24: 100 nF, 50V, X7R, Capacitor_SMD:C_0402_1005Metric, symbol Device:C_Small
- added C25: 1 uF, 16V, X5R, Capacitor_SMD:C_0402_1005Metric, symbol Device:C_Small
- C26: value 5.6 nF, 50V -> 6.8 nF, 50V; LCSC C281760 -> C1542
- Q3, Q5: value Q_PMOS-E_DUAL_Generic_SEP_S1G1D2S2G2D1 -> FDC6306P; footprint PCM_Package_TO_SOT_SMD_AKL:Vishay_PowerPAK_SC70-6L_Dual -> PCM_Package_TO_SOT_SMD_AKL:TSOT-23-6; symbol PCM_Transistor_MOSFET_AKL:Q_PMOS-E_DUAL_Generic_SEP_S1G1D2S2G2D1 -> PCM_Transistor_MOSFET_AKL:Q_PMOS-E_DUAL_Generic_SEP_G1S2G2D2S1D1; LCSC (none) -> C558119
- RN1, RN2: LCSC (none) -> C25725
- U4: footprint W25Q16JVUXIQ:SON50P300X200X60-9N -> ul_W25Q16JVUXIQ:W25Q16JVUXIQ_WIN
Connections:
- net +3V3: now also C24.1, C25.1
- net CIN1: now also CN1.1 (Pin_1); no longer J14.2 (Pin_2)
- net CIN2: now also J14.7 (Pin_7); no longer J14.4 (Pin_4)
- net CIN3: now also J14.5 (Pin_5); no longer J14.7 (Pin_7)
- net CIN4: now also J14.4 (Pin_4); no longer CN1.1 (Pin_1)
- net CN5_DRAIN: now also U16.4 (DRAIN1)
- net CN6_4: now also U15.12 (DRAIN5)
- net CN6_6: now also U15.13 (DRAIN6)
- net CN6_8: now also U15.14 (DRAIN7)
- net CN9_DRAIN: now also U16.3 (DRAIN0)
- net C_SHIELD_1: now also J14.8 (Pin_8)
- net C_SHIELD_2: now also J14.2 (Pin_2), J14.3 (Pin_3); no longer J14.5 (Pin_5)
- net GND: now also C24.2, C25.2; no longer J14.3 (Pin_3), J14.8 (Pin_8)
- net JP2_FA10: now also U15.3 (DRAIN0)
- net JP2_FA7: now also U15.6 (DRAIN3)
- net JP2_FA8: now also U15.5 (DRAIN2)
- net JP2_FA9: now also U15.4 (DRAIN1)
- net VOUT_1: now also Q5.4 (D2); no longer Q5.3 (D2)
- net VOUT_1_GATE: now also Q5.3 (G2); no longer Q5.5 (G2)
- net VOUT_2_GATE: now also Q3.1 (G1); no longer Q3.2 (G1)
- net VOUT_3: now also Q3.4 (D2); no longer Q3.3 (D2)
- net VOUT_3_GATE: now also Q3.3 (G2); no longer Q3.5 (G2)
- net at JP6.2 (C), R30.1: now also Q3.2 (S2); no longer Q3.4 (S2)
- net at JP5.2 (C), R29.1: now also Q3.5 (S1); no longer Q3.1 (S1)
- net at JP4.2 (C), R28.1: now also Q5.2 (S2); no longer Q5.4 (S2)
Other:
- note added: "IO"
- note added: "Originally specced as 5.6 nF Switched to 6.8 nF, because it's available as JLCPCB Basic Part Changes start-up time from 2.8 ms to 3.4 ms"
- note added: "Verified"
- note added: "Very similar to Open LCC"
- note removed: "Espresso IO"
- moved on the sheet: CN5, CN6, CN7, CN9, J1, J13, J5, JP3, JP4, JP5, JP6, Q3A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
