File: open-control-board.kicad_sch (KiCad schematic)
At the start: 123 parts, among them CN1 Service boiler fill sensor, CN10 LCC Port, CN2 Water tank level switch, CN3 NTC Service Boiler, CN4 NTC Brew Boiler, CN5 Service boiler relay, CN6 Conn_02x04_Counter_Clockwise, CN7 Brew Switch, CN8 12V Separate Supply, CN9 Brew boiler relay, J1 USB_B_Micro, J10 Conn_01x04_Pin, J11 Conn_01x04_Pin, J12 Conn_02x06_Odd_Even, J13 Conn_02x05_Odd_Even, J14 Conn_02x04_Odd_Even, J15 Conn_02x05_Odd_Even, J16 USB_B_Micro, J18 Conn_01x03_Pin, J5 BM04B-SRSS-TB(LF)(SN), Q1 AO3401A, Q11 DMN63D8LDW, Q2 AO3401A, Q3 Q_PMOS-E_DUAL_Generic_SEP_S1G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, Q4 DMN63D8LDW, Q5 Q_PMOS-E_DUAL_Generic_SEP_S1G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, Q6 DMN63D8LDW, SW1 SW_Push, SW2 SW_Push, SW3 SW_Push, SW4 SW_Push, U10 FDC1004, U15 STPIC6C595TTR, U16 STPIC6C595TTR, U2 RP2040, U3 ESP32-S3-WROOM-1, U4 W25Q16JVUXIQ, U6 TPS82130, U7 TXB0108PWR, U8 ADS1115IDGS, Y1 XYDBPCNANF-12MHZ

Commit message: Updated project symbols and footprints
Parts:
- CN1, CN10, CN2, CN3, CN4, CN5, CN6, CN7, CN8, CN9, J10, J11, J12, J13, J14, J15, J18, JP13, JP2, JP3, JP4, JP5, JP6, JP7, JP9: now left out of the parts list
- SW1, SW2, SW3, SW4: now in the parts list
Changed lines of the file:
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@@
   )
   (symbol (lib_id "Jumper:SolderJumper_3_Bridged12") (at -82.55 229.87 90) (unit 1)
-    (in_bom yes) (on_board yes) (dnp no) (fields_autoplaced)
+    (in_bom no) (on_board yes) (dnp no) (fields_autoplaced)
     (property "Reference" "JP4" (at -85.09 228.6 90)
       (effects (font (size 1.27 1.27)) (justify left))
@@
   )
   (symbol (lib_id "Switch:SW_Push") (at 40.64 422.91 0) (unit 1)
-    (in_bom no) (on_board yes) (dnp no) (fields_autoplaced)
+    (in_bom yes) (on_board yes) (dnp no) (fields_autoplaced)
     (property "Reference" "SW2" (at 40.64 415.29 0)
       (effects (font (size 1.27 1.27)))
@@
   )
   (symbol (lib_id "Connector:Conn_01x02_Pin") (at 22.86 104.14 0) (unit 1)
-    (in_bom yes) (on_board yes) (dnp no) (fields_autoplaced)
+    (in_bom no) (on_board yes) (dnp no) (fields_autoplaced)
     (property "Reference" "CN5" (at 23.495 99.06 0)
       (effects (font (size 1.27 1.27)))
@@
   )
   (symbol (lib_id "Connector:Conn_01x02_Pin") (at 27.94 71.12 0) (unit 1)
-    (in_bom yes) (on_board yes) (dnp no) (fields_autoplaced)
+    (in_bom no) (on_board yes) (dnp no) (fields_autoplaced)
     (property "Reference" "CN3" (at 28.575 66.04 0)
       (effects (font (size 1.27 1.27)))
@@
   )
   (symbol (lib_id "Connector:Conn_01x02_Pin") (at 26.67 130.81 0) (unit 1)
-    (in_bom yes) (on_board yes) (dnp no) (fields_autoplaced)
+    (in_bom no) (on_board yes) (dnp no) (fields_autoplaced)
     (property "Reference" "CN9" (at 27.305 125.73 0)
       (effects (font (size 1.27 1.27)))
@@
   )
   (symbol (lib_id "Connector_Generic:Conn_02x04_Odd_Even") (at 80.01 81.28 0) (unit 1)
-    (in_bom yes) (on_board yes) (dnp no) (fields_autoplaced)
+    (in_bom no) (on_board yes) (dnp no) (fields_autoplaced)
     (property "Reference" "J14" (at 81.28 72.39 0)
       (effects (font (size 1.27 1.27)))
@@
   )
   (symbol (lib_id "Jumper:SolderJumper_3_Bridged12") (at 307.34 254 0) (mirror y) (unit 1)
-    (in_bom yes) (on_board yes) (dnp no)
+    (in_bom no) (on_board yes) (dnp no)
     (property "Reference" "JP13" (at 309.88 251.46 0)
       (effects (font (size 1.27 1.27)) (justify left))
@@
   )
   (symbol (lib_id "Jumper:SolderJumper_3_Bridged12") (at -82.55 279.4 90) (unit 1)
-    (in_bom yes) (on_board yes) (dnp no) (fields_autoplaced)
+    (in_bom no) (on_board yes) (dnp no) (fields_autoplaced)
     (property "Reference" "JP5" (at -85.09 278.13 90)
       (effects (font (size 1.27 1.27)) (justify left))
@@
   )
   (symbol (lib_id "Switch:SW_Push") (at 40.64 407.67 0) (unit 1)
-    (in_bom no) (on_board yes) (dnp no) (fields_autoplaced)
+    (in_bom yes) (on_board yes) (dnp no) (fields_autoplaced)
     (property "Reference" "SW1" (at 40.64 400.05 0)
       (effects (font (size 1.27 1.27)))
@@
   )
   (symbol (lib_id "Connector_Generic:Conn_02x05_Odd_Even") (at 35.56 223.52 0) (unit 1)
-    (in_bom yes) (on_board yes) (dnp no) (fields_autoplaced)
+    (in_bom no) (on_board yes) (dnp no) (fields_autoplaced)
     (property "Reference" "J13" (at 36.83 212.09 0)
       (effects (font (size 1.27 1.27)))
@@
   )
   (symbol (lib_id "Connector:Conn_01x03_Pin") (at 633.73 49.53 180) (unit 1)
-    (in_bom yes) (on_board yes) (dnp no) (fields_autoplaced)
+    (in_bom no) (on_board yes) (dnp no) (fields_autoplaced)
     (property "Reference" "J18" (at 635 48.26 0)
       (effects (font (size 1.27 1.27)) (justify right))
@@
   )
   (symbol (lib_id "Connector_Generic:Conn_02x05_Odd_Even") (at 501.65 163.83 0) (unit 1)
-    (in_bom yes) (on_board yes) (dnp no) (fields_autoplaced)
+    (in_bom no) (on_board yes) (dnp no) (fields_autoplaced)
     (property "Reference" "J15" (at 502.92 152.4 0)
       (effects (font (size 1.27 1.27)))
@@
   )
   (symbol (lib_id "Switch:SW_Push") (at 520.7 222.25 0) (unit 1)
-    (in_bom no) (on_board yes) (dnp no) (fields_autoplaced)
+    (in_bom yes) (on_board yes) (dnp no) (fields_autoplaced)
     (property "Reference" "SW4" (at 520.7 214.63 0)
       (effects (font (size 1.27 1.27)))
@@
   )
   (symbol (lib_id "Connector:Conn_01x02_Pin") (at 27.94 82.55 0) (unit 1)
-    (in_bom yes) (on_board yes) (dnp no) (fields_autoplaced)
+    (in_bom no) (on_board yes) (dnp no) (fields_autoplaced)
     (property "Reference" "CN4" (at 28.575 77.47 0)
       (effects (font (size 1.27 1.27)))
@@
   )
   (symbol (lib_id "Connector:Conn_01x04_Pin") (at 72.39 31.75 0) (unit 1)
-    (in_bom yes) (on_board yes) (dnp no) (fields_autoplaced)
+    (in_bom no) (on_board yes) (dnp no) (fields_autoplaced)
     (property "Reference" "J10" (at 73.025 24.13 0)
       (effects (font (size 1.27 1.27)))
@@
   )
   (symbol (lib_id "Connector_Generic:Conn_02x04_Odd_Even") (at 34.29 148.59 0) (unit 1)
-    (in_bom yes) (on_board yes) (dnp no) (fields_autoplaced)
+    (in_bom no) (on_board yes) (dnp no) (fields_autoplaced)
     (property "Reference" "CN6" (at 35.56 139.7 0)
       (effects (font (size 1.27 1.27)))
@@
   )
   (symbol (lib_id "Connector:Conn_01x02_Pin") (at 27.94 48.26 0) (unit 1)
-    (in_bom yes) (on_board yes) (dnp no) (fields_autoplaced)
+    (in_bom no) (on_board yes) (dnp no) (fields_autoplaced)
     (property "Reference" "CN1" (at 28.575 43.18 0)
       (effects (font (size 1.27 1.27)))
@@
   )
   (symbol (lib_id "Jumper:SolderJumper_3_Bridged12") (at 34.29 194.31 180) (unit 1)
-    (in_bom yes) (on_board yes) (dnp no) (fields_autoplaced)
+    (in_bom no) (on_board yes) (dnp no) (fields_autoplaced)
     (property "Reference" "JP9" (at 34.29 198.12 0)
       (effects (font (size 1.27 1.27)))
@@
   )
   (symbol (lib_id "Connector:Conn_01x04_Pin") (at 72.39 63.5 0) (unit 1)
-    (in_bom yes) (on_board yes) (dnp no) (fields_autoplaced)
+    (in_bom no) (on_board yes) (dnp no) (fields_autoplaced)
     (property "Reference" "J11" (at 73.025 55.88 0)
       (effects (font (size 1.27 1.27)))
@@
   )
   (symbol (lib_id "Connector:Conn_01x06_Pin") (at 27.94 30.48 0) (unit 1)
-    (in_bom yes) (on_board yes) (dnp no) (fields_autoplaced)
+    (in_bom no) (on_board yes) (dnp no) (fields_autoplaced)
     (property "Reference" "JP2" (at 28.575 20.32 0)
       (effects (font (size 1.27 1.27)))
@@
   )
   (symbol (lib_id "Connector_Generic:Conn_02x06_Odd_Even") (at 74.93 105.41 0) (unit 1)
-    (in_bom yes) (on_board yes) (dnp no) (fields_autoplaced)
+    (in_bom no) (on_board yes) (dnp no) (fields_autoplaced)
     (property "Reference" "J12" (at 76.2 93.98 0)
       (effects (font (size 1.27 1.27)))
@@
   )
   (symbol (lib_id "Jumper:Jumper_2_Open") (at 563.88 165.1 90) (unit 1)
-    (in_bom yes) (on_board yes) (dnp no) (fields_autoplaced)
+    (in_bom no) (on_board yes) (dnp no) (fields_autoplaced)
     (property "Reference" "JP7" (at 565.15 163.83 90)
       (effects (font (size 1.27 1.27)) (justify right))
@@
   )
   (symbol (lib_id "Jumper:SolderJumper_3_Bridged12") (at -82.55 325.12 90) (unit 1)
-    (in_bom yes) (on_board yes) (dnp no) (fields_autoplaced)
+    (in_bom no) (on_board yes) (dnp no) (fields_autoplaced)
     (property "Reference" "JP6" (at -85.09 323.85 90)
       (effects (font (size 1.27 1.27)) (justify left))
@@
   )
   (symbol (lib_id "Connector:Conn_01x06_Pin") (at 22.86 172.72 0) (unit 1)
-    (in_bom yes) (on_board yes) (dnp no) (fields_autoplaced)
+    (in_bom no) (on_board yes) (dnp no) (fields_autoplaced)
     (property "Reference" "CN10" (at 23.495 162.56 0)
       (effects (font (size 1.27 1.27)))
@@
   )
   (symbol (lib_id "Switch:SW_Push") (at 520.7 207.01 0) (unit 1)
-    (in_bom no) (on_board yes) (dnp no) (fields_autoplaced)
+    (in_bom yes) (on_board yes) (dnp no) (fields_autoplaced)
     (property "Reference" "SW3" (at 520.7 199.39 0)
       (effects (font (size 1.27 1.27)))
@@
   )
   (symbol (lib_id "Connector:Conn_01x02_Pin") (at 26.67 119.38 0) (unit 1)
-    (in_bom yes) (on_board yes) (dnp no) (fields_autoplaced)
+    (in_bom no) (on_board yes) (dnp no) (fields_autoplaced)
     (property "Reference" "CN7" (at 27.305 114.3 0)
       (effects (font (size 1.27 1.27)))
@@
   )
   (symbol (lib_id "Jumper:Jumper_2_Open") (at 40.64 254 90) (unit 1)
-    (in_bom yes) (on_board yes) (dnp no) (fields_autoplaced)
+    (in_bom no) (on_board yes) (dnp no) (fields_autoplaced)
     (property "Reference" "JP3" (at 41.91 252.73 90)
       (effects (font (size 1.27 1.27)) (justify right))
@@
   )
   (symbol (lib_id "Connector:Conn_01x02_Pin") (at 27.94 59.69 0) (unit 1)
-    (in_bom yes) (on_board yes) (dnp no) (fields_autoplaced)
+    (in_bom no) (on_board yes) (dnp no) (fields_autoplaced)
     (property "Reference" "CN2" (at 28.575 54.61 0)
       (effects (font (size 1.27 1.27)))
@@
   )
   (symbol (lib_id "Connector:Conn_01x02_Pin") (at 72.39 48.26 0) (unit 1)
-    (in_bom yes) (on_board yes) (dnp no) (fields_autoplaced)
+    (in_bom no) (on_board yes) (dnp no) (fields_autoplaced)
     (property "Reference" "CN8" (at 73.025 43.18 0)
       (effects (font (size 1.27 1.27)))
