File: open-control-board.kicad_sch (KiCad schematic)
At the start: 199 parts, among them CN1 LCC Port, CN14 Conn_02x06_Odd_Even, CN2 Conn_01x06_Pin, CN3 12V Separate Supply, CN4 Conn_02x05_Counter_Clockwise, CN5 NTC Brew Boiler, CN6 NTC Service Boiler, CN7 Conn_01x06_Pin, CN8 Conn_01x05_Pin, J1 USB_B_Micro, J13 Conn_02x05_Odd_Even, J15 Conn_02x05_Odd_Even, J16 USB_B_Micro, J3 Conn_02x03_Odd_Even, J4 Molex_0525591853, J5 BM04B-SRSS-TB(LF)(SN), J5 Micro_SD_Card_Det_Hirose_DM3AT, Q1 DMP21D0UT-7, Q10 DMG1012T-7, Q11 DMN63D8LDW, Q12 DMN63D8LDW, Q13 DMG1012T-7, Q14 DMG1012T-7, Q15 DMP21D0UT-7, Q16 DMG1012T-7, Q2 DMP21D0UT-7, Q3 Q_PMOS-E_DUAL_Generic_SEP_S1G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, Q4 DMN63D8LDW, Q5 Q_PMOS-E_DUAL_Generic_SEP_S1G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, Q6 DMN63D8LDW, Q7 DMN63D8LDW, Q8 DMP21D0UT-7, Q9 DMG1012T-7, SW1 SW_Push, SW2 SW_Push, SW3 SW_Push, SW4 SW_Push, U10 FDC1004, U11 TC2014-5.0VxCTTR, U15 STPIC6C595TTR, U16 STPIC6C595TTR, U2 RP2040, U3 ESP32-S3-WROOM-1, U4 W25Q16JVUXIQ, U6 ADS124S08IPBSR, U6 TPS82130, U7 LM5050-1, U8 LM5050-1, Y1 XYDBPCNANF-12MHZ

Commit message: Fixes
Connections:
- net CN14_6_3V3 is gone; now on net CN14_8: JP15.1 (A)
- net +3V3: now also U6.15 (IOVDD)
- net ESP32_U0RXD: now also J3.5 (Pin_5); no longer J3.3 (Pin_3)
- net ESP32_U0TXD: now also J3.3 (Pin_3); no longer J3.5 (Pin_5)
- net GND: now also C47.2, U6.24 (REFCOM); no longer U6.15 (IOVDD)
- net QWIIC_SDA: now also U15.11 (DRAIN4)
- no-connect marks 20 -> 19
Other:
- note added: "By connecting this to SDA, we can do a self- diagnostic on boot-up"
Changed lines of the file:
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@@
   (junction (at 330.2 46.99) (diameter 0) (color 0 0 0 0)
   )
+  (junction (at 902.97 46.99) (diameter 0) (color 0 0 0 0)
+  )
   (junction (at 196.85 198.12) (diameter 0) (color 0 0 0 0)
   )
@@
   (junction (at 36.83 355.6) (diameter 0) (color 0 0 0 0)
   )
-  (junction (at 905.51 95.25) (diameter 0) (color 0 0 0 0)
-  )
   (junction (at 529.59 285.75) (diameter 0) (color 0 0 0 0)
   )
@@
   (junction (at 280.67 160.02) (diameter 0) (color 0 0 0 0)
   )
+  (junction (at 905.51 100.33) (diameter 0) (color 0 0 0 0)
+  )
   (junction (at 224.79 27.94) (diameter 0) (color 0 0 0 0)
   )
@@
   (junction (at 905.51 107.95) (diameter 0) (color 0 0 0 0)
   )
+  (junction (at 905.51 95.25) (diameter 0) (color 0 0 0 0)
+  )
   (junction (at 274.32 279.4) (diameter 0) (color 0 0 0 0)
   )
@@
   (junction (at 1123.95 170.18) (diameter 0) (color 0 0 0 0)
   )
-  (junction (at 905.51 100.33) (diameter 0) (color 0 0 0 0)
-  )
   (junction (at 311.15 510.54) (diameter 0) (color 0 0 0 0)
   )
@@
   (no_connect (at 899.16 90.17))
   (no_connect (at 514.35 118.11))
-  (no_connect (at 187.96 152.4))
   (no_connect (at 899.16 59.69))
   (no_connect (at 187.96 223.52))
@@
     (stroke (width 0) (type default))
   )
+  (wire (pts (xy 905.51 106.68) (xy 905.51 107.95))
+    (stroke (width 0) (type default))
+  )
   (wire (pts (xy 619.76 179.07) (xy 612.14 179.07))
     (stroke (width 0) (type default))
@@
     (stroke (width 0) (type default))
   )
+  (wire (pts (xy 905.51 95.25) (xy 908.05 95.25))
+    (stroke (width 0) (type default))
+  )
   (wire (pts (xy 774.7 203.2) (xy 774.7 204.47))
     (stroke (width 0) (type default))
@@
     (stroke (width 0) (type default))
   )
+  (wire (pts (xy 905.51 95.25) (xy 905.51 100.33))
+    (stroke (width 0) (type default))
+  )
   (wire (pts (xy 354.33 203.2) (xy 354.33 187.96))
     (stroke (width 0) (type default))
@@
     (stroke (width 0) (type default))
   )
-  (wire (pts (xy 905.51 100.33) (xy 905.51 107.95))
+  (wire (pts (xy 905.51 100.33) (xy 905.51 101.6))
     (stroke (width 0) (type default))
   )
@@
     (stroke (width 0) (type default))
   )
-  (wire (pts (xy 908.05 95.25) (xy 905.51 95.25))
-    (stroke (width 0) (type default))
-  )
   (wire (pts (xy 292.1 393.7) (xy 297.18 393.7))
     (stroke (width 0) (type default))
@@
     (stroke (width 0) (type default))
   )
-  (wire (pts (xy 905.51 95.25) (xy 899.16 95.25))
+  (wire (pts (xy 899.16 95.25) (xy 905.51 95.25))
     (stroke (width 0) (type default))
   )
@@
     (stroke (width 0) (type default))
   )
+  (wire (pts (xy 187.96 152.4) (xy 218.44 152.4))
+    (stroke (width 0) (type default))
+  )
   (wire (pts (xy 568.96 181.61) (xy 575.31 181.61))
     (stroke (width 0) (type default))
@@
     (effects (font (size 1.27 1.27)) (justify left bottom))
   )
+  (text "By connecting this to SDA, \nwe can do a self-\ndiagnostic on boot-up"
+    (at 217.17 160.02 0)
+    (effects (font (size 1.27 1.27)) (justify left bottom))
+  )
   (text "EyeSPI Connector" (at 709.93 86.36 0)
     (effects (font (size 1.27 1.27)) (justify left bottom))
@@
     )
   )
-  (global_label "ESP32_U0RXD" (shape input) (at 496.57 186.69 180) (fields_autoplaced)
-    (effects (font (size 1.27 1.27)) (justify right))
-    (property "Intersheetrefs" "${INTERSHEET_REFS}" (at 480.2802 186.69 0)
-      (effects (font (size 1.27 1.27)) (justify right) hide)
-    )
-  )
   (global_label "CN1_UART_RX_SHIFT_SEL" (shape output) (at 300.99 330.2 0) (fields_autoplaced)
     (effects (font (size 1.27 1.27)) (justify left))
@@
     )
   )
+  (global_label "ESP32_U0TXD" (shape output) (at 496.57 186.69 180) (fields_autoplaced)
+    (effects (font (size 1.27 1.27)) (justify right))
+    (property "Intersheetrefs" "${INTERSHEET_REFS}" (at 480.5826 186.69 0)
+      (effects (font (size 1.27 1.27)) (justify right) hide)
+    )
+  )
   (global_label "INT_SPI_MOSI" (shape output) (at 379.73 152.4 0) (fields_autoplaced)
     (effects (font (size 1.27 1.27)) (justify left))
@@
     )
   )
-  (global_label "CN14_6_3V3" (shape bidirectional) (at 679.45 234.95 180) (fields_autoplaced)
+  (global_label "CN14_8" (shape bidirectional) (at 679.45 234.95 180) (fields_autoplaced)
     (effects (font (size 1.27 1.27)) (justify right))
-    (property "Intersheetrefs" "${INTERSHEET_REFS}" (at 665.9193 234.95 0)
-      (effects (font (size 1.27 1.27)) (justify right) hide)
-    )
-  )
-  (global_label "ESP32_U0TXD" (shape output) (at 496.57 189.23 180) (fields_autoplaced)
-    (effects (font (size 1.27 1.27)) (justify right))
-    (property "Intersheetrefs" "${INTERSHEET_REFS}" (at 480.5826 189.23 0)
+    (property "Intersheetrefs" "${INTERSHEET_REFS}" (at 668.1569 234.95 0)
       (effects (font (size 1.27 1.27)) (justify right) hide)
     )
@@
     )
   )
+  (global_label "ESP32_U0RXD" (shape input) (at 496.57 189.23 180) (fields_autoplaced)
+    (effects (font (size 1.27 1.27)) (justify right))
+    (property "Intersheetrefs" "${INTERSHEET_REFS}" (at 480.2802 189.23 0)
+      (effects (font (size 1.27 1.27)) (justify right) hide)
+    )
+  )
   (global_label "ESP32_EN" (shape input) (at 509.27 168.91 0) (fields_autoplaced)
     (effects (font (size 1.27 1.27)) (justify left))
@@
     )
   )
+  (global_label "QWIIC_SDA" (shape bidirectional) (at 218.44 152.4 0) (fields_autoplaced)
+    (effects (font (size 1.27 1.27)) (justify left))
+    (property "Intersheetrefs" "${INTERSHEET_REFS}" (at 232.3337 152.4 0)
+      (effects (font (size 1.27 1.27)) (justify left) hide)
+    )
+  )
   (global_label "CN12_HighI" (shape bidirectional) (at 307.34 576.58 0) (fields_autoplaced)
     (effects (font (size 1.27 1.27)) (justify left))
@@
     )
   )
+  (symbol (lib_id "power:GNDA") (at 902.97 46.99 0) (unit 1)
+    (in_bom yes) (on_board yes) (dnp no) (fields_autoplaced)
+    (property "Reference" "#PWR0186" (at 902.97 53.34 0)
+      (effects (font (size 1.27 1.27)) hide)
+    )
+    (property "Value" "GNDA" (at 902.97 52.07 0)
+      (effects (font (size 1.27 1.27)))
+    )
+    (property "Footprint" "" (at 902.97 46.99 0)
+      (effects (font (size 1.27 1.27)) hide)
+    )
+    (property "Datasheet" "" (at 902.97 46.99 0)
+      (effects (font (size 1.27 1.27)) hide)
+    )
+    (pin "1")
+    (instances
+      (project "open-control-board"
+        (path "/c7c8c763-88fa-419b-8f4a-ebade330cc39"
+          (reference "#PWR0186") (unit 1)
+        )
+      )
+    )
+  )
   (symbol (lib_id "Jumper:SolderJumper_2_Bridged") (at 1008.38 83.82 90) (unit 1)
     (in_bom no) (on_board yes) (dnp no) (fields_autoplaced)
@@
     )
   )
+  (symbol (lib_id "Device:C_Small") (at 905.51 104.14 0) (unit 1)
+    (in_bom yes) (on_board yes) (dnp no) (fields_autoplaced)
+    (property "Reference" "C45" (at 908.05 102.8763 0)
+      (effects (font (size 1.27 1.27)) (justify left))
+    )
+    (property "Value" "100 nF, >10V, X6S" (at 908.05 105.4163 0)
+      (effects (font (size 1.27 1.27)) (justify left))
+    )
+    (property "Footprint" "Capacitor_SMD:C_0201_0603Metric" (at 905.51 104.14 0)
+      (effects (font (size 1.27 1.27)) hide)
+    )
+    (property "Datasheet" "~" (at 905.51 104.14 0)
+      (effects (font (size 1.27 1.27)) hide)
+    )
+    (property "LCSC" "C412246" (at 905.51 104.14 0)
+      (effects (font (size 1.27 1.27)) hide)
+    )
+    (pin "1")
+    (pin "2")
+    (instances
+      (project "open-control-board"
+        (path "/c7c8c763-88fa-419b-8f4a-ebade330cc39"
+          (reference "C45") (unit 1)
+        )
+      )
+    )
+  )
   (symbol (lib_id "power:+3V3") (at 659.13 189.23 180) (unit 1)
     (in_bom yes) (on_board yes) (dnp no) (fields_autoplaced)
@@
         )
       )
-    )
-  )
-  (symbol (lib_id "Device:C_Small") (at 905.51 97.79 0) (unit 1)
-    (in_bom yes) (on_board yes) (dnp no) (fields_autoplaced)
-    (property "Reference" "C45" (at 908.05 96.5263 0)
-      (effects (font (size 1.27 1.27)) (justify left))
-    )
-    (property "Value" "100 nF, >10V, X6S" (at 908.05 99.0663 0)
-      (effects (font (size 1.27 1.27)) (justify left))
-    )
-    (property "Footprint" "Capacitor_SMD:C_0201_0603Metric" (at 905.51 97.79 0)
-      (effects (font (size 1.27 1.27)) hide)
-    )
-    (property "Datasheet" "~" (at 905.51 97.79 0)
-      (effects (font (size 1.27 1.27)) hide)
-    )
-    (property "LCSC" "C412246" (at 905.51 97.79 0)
-      (effects (font (size 1.27 1.27)) hide)
-    )
-    (pin "1")
-    (pin "2")
-    (instances
-      (project "open-control-board"
-        (path "/c7c8c763-88fa-419b-8f4a-ebade330cc39"
-          (reference "C45") (unit 1)
-        )
-      )
